Commit message: update: versión final de la tesis

File: modelo_scorbot_gazebo/src/scorbot_tf/urdf/scorbot.urdf.xacro (robot description, xacro)
@@ -47,5 +47,16 @@
   <xacro:property name="gripper_upper_limit" value="0.016" />
   <xacro:property name="gripper_lower_limit" value="-0.018" />
-  <xacro:if value="$(arg fixed)">
+ <!--
+   <xacro:property name="fixed" value="true"/>
+   <xacro:if value="${fixed}">
+     <link name="world"/>
+     <joint name="fixed" type="fixed">
+       <parent link="world"/>
+       <child link="base_link"/>
+      </joint>
+    </xacro:if>
+-->
+<!--
+    <xacro:if value="$(arg fixed)">
     <link name="world"/>
     <joint name="fixed" type="fixed">
@@ -54,4 +65,5 @@
     </joint>
   </xacro:if>
+-->
   <link
     name="base_link">
